File: 2chip-16MB-SOJ/MacIIfxRAMSIMM.kicad_pcb (KiCad board)
At the start: 4 copper layers, 97.8 x 25.4 mm, 48 parts, among them J1 IIfxRAM, U1 KM44C16104, U10 XC6206PxxxMR, U2 KM44C16104, U3 74AHCT244PW, U4 74AHCT244PW, U5 74LVC1G04GW, U6 74LVC1G04GW, U7 74LVC1G08GW, U8 74LVC1G74DC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

Commit message: Fabbed
Parts:
- R13: value 100 -> CASd
- R14: value 100 -> CAS
- R15: value 100 -> RCAS
- R16: value 100 -> RCASd
Changed lines of the file:
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@@
   (general
     (thickness 1.6)
-    (drawings 22)
+    (drawings 24)
     (tracks 1059)
     (zones 0)
@@
     (add_net "Net-(U2-Pad7)")
   )
+  (module stdpads:NXP_TSSOP-8_3x3mm_P0.65mm (layer F.Cu)
+    (at 76 109.75)
+    (tags "SSOP-8 MSOP-8")
+    (solder_mask_margin 0.0363)
+    (solder_paste_margin -0.04)
+    (attr smd)
+    (fp_text reference U8 (at 0 0 90) (layer F.Fab)
+      (effects (font (size 0.508 0.508) (thickness 0.127)))
+    )
+    (fp_text value 74LVC1G74DC (at 0 1.3) (layer F.Fab)
+      (effects (font (size 0.127 0.127) (thickness 0.03175)))
+    )
+    (fp_line (start -2 -1.6) (end 1.3 -1.6) (layer F.SilkS) (width 0.127))
+    (fp_line (start -1.5 1.5) (end -1.5 -1.5) (layer F.Fab) (width 0.1))
+    (fp_line (start 1.3 1.6) (end -1.3 1.6) (layer F.SilkS) (width 0.127))
+    (fp_line (start 1.5 -1.5) (end 1.5 1.5) (layer F.Fab) (width 0.1))
+    (fp_line (start -1.5 -1.5) (end 1.5 -1.5) (layer F.Fab) (width 0.1))
+    (fp_line (start 1.5 1.5) (end -1.5 1.5) (layer F.Fab) (width 0.1))
+    (fp_line (start 2.6 1.8) (end 2.6 -1.8) (layer F.CrtYd) (width 0.05))
+    (fp_line (start -2.6 1.8) (end -2.6 -1.8) (layer F.CrtYd) (width 0.05))
+    (fp_line (start -2.6 1.8) (end 2.6 1.8) (layer F.CrtYd) (width 0.05))
+    (fp_line (start -2.6 -1.8) (end 2.6 -1.8) (layer F.CrtYd) (width 0.05))
+    (pad 8 smd roundrect (at 1.65 -1.05) (size 1.15 0.6) (layers F.Cu F.Paste F.Mask) (roundrect_rratio 0.25)
+      (net 25 +3V3))
+    (pad 7 smd roundrect (at 1.65 -0.325) (size 1.15 0.45) (layers F.Cu F.Paste F.Mask) (roundrect_rratio 0.25)
+      (net 25 +3V3))
+    (pad 6 smd roundrect (at 1.65 0.325) (size 1.15 0.45) (layers F.Cu F.Paste F.Mask) (roundrect_rratio 0.25)
+      (net 72 /CAS))
+    (pad 5 smd roundrect (at 1.65 1.05) (size 1.15 0.6) (layers F.Cu F.Paste F.Mask) (roundrect_rratio 0.25)
+      (net 69 /Din~OE~))
+    (pad 4 smd roundrect (at -1.65 1.05) (size 1.15 0.6) (layers F.Cu F.Paste F.Mask) (roundrect_rratio 0.25)
+      (net 7 GND))
+    (pad 3 smd roundrect (at -1.65 0.325) (size 1.15 0.4) (layers F.Cu F.Paste F.Mask) (roundrect_rratio 0.25)
+      (net 70 /Dout~OE~))
+    (pad 2 smd roundrect (at -1.65 -0.325) (size 1.15 0.4) (layers F.Cu F.Paste F.Mask) (roundrect_rratio 0.25)
+      (net 73 /RD))
+    (pad 1 smd roundrect (at -1.65 -1.05) (size 1.15 0.6) (layers F.Cu F.Paste F.Mask) (roundrect_rratio 0.25)
+      (net 82 /CASd))
+    (model ${KISYS3DMOD}/Package_SO.3dshapes/MSOP-8_3x3mm_P0.65mm.wrl
+      (at (xyz 0 0 0))
+      (scale (xyz 0.85 1 1))
+      (rotate (xyz 0 0 0))
+    )
+  )
   (module stdpads:C_0805 (layer F.Cu)
     (at 95.885 119.087 270)
@@
       (effects (font (size 0.254 0.254) (thickness 0.0635)))
     )
-    (fp_text value 100 (at 0 0.35) (layer F.Fab)
+    (fp_text value RCASd (at 0 0.35) (layer F.Fab)
       (effects (font (size 0.254 0.254) (thickness 0.0635)))
     )
@@
       (effects (font (size 0.254 0.254) (thickness 0.0635)))
     )
-    (fp_text value 100 (at 0 0.35) (layer F.Fab)
+    (fp_text value RCAS (at 0 0.35) (layer F.Fab)
       (effects (font (size 0.254 0.254) (thickness 0.0635)))
     )
@@
       (effects (font (size 0.254 0.254) (thickness 0.0635)))
     )
-    (fp_text value 100 (at 0 0.35 90) (layer F.Fab)
+    (fp_text value CAS (at 0 0.35 90) (layer F.Fab)
       (effects (font (size 0.254 0.254) (thickness 0.0635)))
     )
@@
       (effects (font (size 0.254 0.254) (thickness 0.0635)))
     )
-    (fp_text value 100 (at 0 0.35 90) (layer F.Fab)
+    (fp_text value CASd (at 0 0.35 90) (layer F.Fab)
       (effects (font (size 0.254 0.254) (thickness 0.0635)))
     )
@@
       (scale (xyz 1 1 1))
       (rotate (xyz 0 0 -90))
-    )
-  )
-  (module stdpads:NXP_TSSOP-8_3x3mm_P0.65mm (layer F.Cu)
-    (at 76 109.75)
-    (tags "SSOP-8 MSOP-8")
-    (solder_mask_margin 0.04)
-    (solder_paste_margin -0.04)
-    (attr smd)
-    (fp_text reference U8 (at 0 0 90) (layer F.Fab)
-      (effects (font (size 0.508 0.508) (thickness 0.127)))
-    )
-    (fp_text value 74LVC1G74DC (at 0 1.3) (layer F.Fab)
-      (effects (font (size 0.127 0.127) (thickness 0.03175)))
-    )
-    (fp_line (start -2.6 -1.8) (end 2.6 -1.8) (layer F.CrtYd) (width 0.05))
-    (fp_line (start -2.6 1.8) (end 2.6 1.8) (layer F.CrtYd) (width 0.05))
-    (fp_line (start -2.6 1.8) (end -2.6 -1.8) (layer F.CrtYd) (width 0.05))
-    (fp_line (start 2.6 1.8) (end 2.6 -1.8) (layer F.CrtYd) (width 0.05))
-    (fp_line (start 1.5 1.5) (end -1.5 1.5) (layer F.Fab) (width 0.1))
-    (fp_line (start -1.5 -1.5) (end 1.5 -1.5) (layer F.Fab) (width 0.1))
-    (fp_line (start 1.5 -1.5) (end 1.5 1.5) (layer F.Fab) (width 0.1))
-    (fp_line (start 1.3 1.6) (end -1.3 1.6) (layer F.SilkS) (width 0.127))
-    (fp_line (start -1.5 1.5) (end -1.5 -1.5) (layer F.Fab) (width 0.1))
-    (fp_line (start -2 -1.6) (end 1.3 -1.6) (layer F.SilkS) (width 0.127))
-    (pad 1 smd roundrect (at -1.65 -1.05) (size 1.15 0.6) (layers F.Cu F.Paste F.Mask) (roundrect_rratio 0.25)
-      (net 82 /CASd))
-    (pad 2 smd roundrect (at -1.65 -0.325) (size 1.15 0.4) (layers F.Cu F.Paste F.Mask) (roundrect_rratio 0.25)
-      (net 73 /RD))
-    (pad 3 smd roundrect (at -1.65 0.325) (size 1.15 0.4) (layers F.Cu F.Paste F.Mask) (roundrect_rratio 0.25)
-      (net 70 /Dout~OE~))
-    (pad 4 smd roundrect (at -1.65 1.05) (size 1.15 0.6) (layers F.Cu F.Paste F.Mask) (roundrect_rratio 0.25)
-      (net 7 GND))
-    (pad 5 smd roundrect (at 1.65 1.05) (size 1.15 0.6) (layers F.Cu F.Paste F.Mask) (roundrect_rratio 0.25)
-      (net 69 /Din~OE~))
-    (pad 6 smd roundrect (at 1.65 0.325) (size 1.15 0.45) (layers F.Cu F.Paste F.Mask) (roundrect_rratio 0.25)
-      (net 72 /CAS))
-    (pad 7 smd roundrect (at 1.65 -0.325) (size 1.15 0.45) (layers F.Cu F.Paste F.Mask) (roundrect_rratio 0.25)
-      (net 25 +3V3))
-    (pad 8 smd roundrect (at 1.65 -1.05) (size 1.15 0.6) (layers F.Cu F.Paste F.Mask) (roundrect_rratio 0.25)
-      (net 25 +3V3))
-    (model ${KISYS3DMOD}/Package_SO.3dshapes/MSOP-8_3x3mm_P0.65mm.wrl
-      (at (xyz 0 0 0))
-      (scale (xyz 0.85 1 1))
-      (rotate (xyz 0 0 0))
     )
   )
@@
       (net 7 GND) (zone_connect 2))
   )
+  (gr_poly (pts (xy 163.195 127.635) (xy 123.825 127.635) (xy 123.317 125.0315) (xy 163.703 125.0315)) (layer B.Mask) (width 0.175))
+  (gr_poly (pts (xy 117.475 127.635) (xy 78.105 127.635) (xy 77.597 125.0315) (xy 117.983 125.0315)) (layer B.Mask) (width 0.175))
   (gr_text "ZK,\nGF" (at 165.354 125.603) (layer B.SilkS)
     (effects (font (size 0.8128 0.8128) (thickness 0.2032)) (justify mirror))
@@
   (segment (start 140.3495 122.555) (end 140.3495 123.4585) (width 0.5) (layer F.Cu) (net 7))
   (via (at 137.7315 122.7455) (size 0.5) (drill 0.2) (layers F.Cu B.Cu) (net 7))
-  (segment (start 75.95 107.75) (end 76.1 107.9) (width 0.6) (layer F.Cu) (net 7))
-  (via (at 76.1 107.9) (size 0.6) (drill 0.3) (layers F.Cu B.Cu) (net 7))
-  (segment (start 75.95 106.8) (end 75.95 107.75) (width 0.6) (layer F.Cu) (net 7))
+  (via (at 75.9 107.9) (size 0.6) (drill 0.3) (layers F.Cu B.Cu) (net 7))
   (via (at 76.1 105.7) (size 0.5) (drill 0.2) (layers F.Cu B.Cu) (net 7))
   (segment (start 75.95 105.85) (end 76.1 105.7) (width 0.5) (layer F.Cu) (net 7))
@@
   (via (at 159.512 116.0145) (size 0.5) (drill 0.2) (layers F.Cu B.Cu) (net 7))
   (via (at 151.8285 116.078) (size 0.5) (drill 0.2) (layers F.Cu B.Cu) (net 7))
+  (segment (start 75.95 107.85) (end 75.9 107.9) (width 0.6) (layer F.Cu) (net 7))
+  (segment (start 75.95 106.8) (end 75.95 107.85) (width 0.6) (layer F.Cu) (net 7))
   (segment (start 125.095 118.442) (end 125.095 120.904) (width 0.15) (layer F.Cu) (net 8))
   (segment (start 125.095 120.904) (end 122.8725 123.1265) (width 0.15) (layer F.Cu) (net 8))
