File: 2chip-16MB-SOJ/MacIIfxRAMSIMM.sch (KiCad schematic (older format))
At the start: 48 parts, among them J1 IIfxRAM, U1 KM44C16104, U10 XC6206PxxxMR, U2 KM44C16104, U3 74AHCT244PW, U4 74AHCT244PW, U5 74LVC1G04GW, U6 74LVC1G04GW, U7 74LVC1G08GW, U8 74LVC1G74DC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

Commit message: Fabbed
Parts:
- R13: value 100 -> CASd
- R14: value 100 -> CAS
- R15: value 100 -> RCAS
- R16: value 100 -> RCASd
Other:
- moved on the sheet: R15, R16
Changed lines of the file:
@@
 P 6750 850
 F 0 "R13" V 6600 850 50  0000 C CNN
-F 1 "100" V 6700 850 50  0000 C BNN
+F 1 "CASd" V 6700 850 50  0000 C BNN
 F 2 "stdpads:R_0805" H 6750 850 50  0001 C CNN
 F 3 "~" H 6750 850 50  0001 C CNN
@@
 P 6750 1150
 F 0 "R14" V 6600 1150 50  0000 C CNN
-F 1 "100" V 6700 1150 50  0000 C BNN
+F 1 "CAS" V 6700 1150 50  0000 C BNN
 F 2 "stdpads:R_0805" H 6750 1150 50  0001 C CNN
 F 3 "~" H 6750 1150 50  0001 C CNN
@@
 Text Label 7400 1000 0    50   ~ 0
 ~CAS~d
-Wire Wire Line
-	7400 1000 7600 1000
-$Comp
-L Device:R_Small R15
-U 1 1 6121B08E
-P 7700 700
-F 0 "R15" V 7550 700 50  0000 C CNN
-F 1 "100" V 7650 700 50  0000 C BNN
-F 2 "stdpads:R_0805" H 7700 700 50  0001 C CNN
-F 3 "~" H 7700 700 50  0001 C CNN
-	1    7700 700
-	0    -1   1    0
-$EndComp
-$Comp
-L Device:R_Small R16
-U 1 1 6121B094
-P 7700 1000
-F 0 "R16" V 7550 1000 50  0000 C CNN
-F 1 "100" V 7650 1000 50  0000 C BNN
-F 2 "stdpads:R_0805" H 7700 1000 50  0001 C CNN
-F 3 "~" H 7700 1000 50  0001 C CNN
-	1    7700 1000
-	0    -1   1    0
-$EndComp
-Wire Wire Line
-	7800 700  7800 1000
-Text Label 8000 1000 2    50   ~ 0
-R~CAS~
-Wire Wire Line
-	8000 1000 7800 1000
-Connection ~ 7800 1000
 Text Label 7400 700  0    50   ~ 0
 ~CAS~
-Wire Wire Line
-	7400 700  7600 700
 $Comp
 L power:GND #PWR0137
@@
 	1    0    0    -1
 $EndComp
+Wire Wire Line
+	7900 700  7900 1000
+Text Label 8100 1000 2    50   ~ 0
+R~CAS~
+Wire Wire Line
+	7900 1000 7850 1000
+Wire Wire Line
+	7400 1000 7650 1000
+Wire Wire Line
+	7400 700  7650 700
+Wire Wire Line
+	7900 1000 8100 1000
+Connection ~ 7900 1000
+$Comp
+L Device:R_Small R16
+U 1 1 6121B094
+P 7750 1000
+F 0 "R16" V 7600 1000 50  0000 C CNN
+F 1 "RCASd" V 7700 1000 50  0000 C BNN
+F 2 "stdpads:R_0805" H 7750 1000 50  0001 C CNN
+F 3 "~" H 7750 1000 50  0001 C CNN
+	1    7750 1000
+	0    -1   1    0
+$EndComp
+$Comp
+L Device:R_Small R15
+U 1 1 6121B08E
+P 7750 700
+F 0 "R15" V 7600 700 50  0000 C CNN
+F 1 "RCAS" V 7700 700 50  0000 C BNN
+F 2 "stdpads:R_0805" H 7750 700 50  0001 C CNN
+F 3 "~" H 7750 700 50  0001 C CNN
+	1    7750 700
+	0    -1   1    0
+$EndComp
+Wire Wire Line
+	7900 700  7850 700
 $EndSCHEMATC
