File: 2chip-16MB-SOP/MacIIfxRAMSIMM.kicad_pcb (KiCad board)
At the start: 4 copper layers, 97.8 x 25.4 mm, 48 parts, among them J1 IIfxRAM, U1 KM44C16104, U10 XC6206PxxxMR, U2 KM44C16104, U3 74AHCT244PW, U4 74AHCT244PW, U5 74LVC1G04GW, U6 74LVC1G04GW, U7 74LVC1G08GW, U8 74LVC1G74DC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

Commit message: Fabbed
Parts:
- R13: value 100 -> CASd
- R14: value 100 -> CAS
- R15: value 100 -> RCAS
- R16: value 100 -> RCASd
