File: Adapter-30/Adapter-30.kicad_sch (KiCad schematic)
At the start: 12 parts, among them J1 DRAM-SIMM-30, J2 IIfxRAM

Commit message: Prototype adapter-30
Parts:
- removed C5, C6: 2u2, stdpads:C_0805, symbol Device:C_Small
Changed lines of the file:
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@@
   (junction (at 132.08 62.23) (diameter 0) (color 0 0 0 0)
   )
+  (junction (at 132.08 57.15) (diameter 0) (color 0 0 0 0)
+  )
+  (junction (at 132.08 54.61) (diameter 0) (color 0 0 0 0)
+  )
+  (junction (at 93.98 161.29) (diameter 0) (color 0 0 0 0)
+  )
+  (junction (at 132.08 67.31) (diameter 0) (color 0 0 0 0)
+  )
+  (junction (at 132.08 69.85) (diameter 0) (color 0 0 0 0)
+  )
+  (junction (at 215.9 34.29) (diameter 0) (color 0 0 0 0)
+  )
+  (junction (at 93.98 156.21) (diameter 0) (color 0 0 0 0)
+  )
+  (junction (at 203.2 71.12) (diameter 0) (color 0 0 0 0)
+  )
+  (junction (at 132.08 59.69) (diameter 0) (color 0 0 0 0)
+  )
   (junction (at 104.14 161.29) (diameter 0) (color 0 0 0 0)
-  )
-  (junction (at 132.08 57.15) (diameter 0) (color 0 0 0 0)
-  )
-  (junction (at 132.08 54.61) (diameter 0) (color 0 0 0 0)
-  )
-  (junction (at 93.98 161.29) (diameter 0) (color 0 0 0 0)
-  )
-  (junction (at 132.08 67.31) (diameter 0) (color 0 0 0 0)
-  )
-  (junction (at 114.3 156.21) (diameter 0) (color 0 0 0 0)
-  )
-  (junction (at 104.14 156.21) (diameter 0) (color 0 0 0 0)
-  )
-  (junction (at 124.46 161.29) (diameter 0) (color 0 0 0 0)
-  )
-  (junction (at 132.08 69.85) (diameter 0) (color 0 0 0 0)
-  )
-  (junction (at 114.3 161.29) (diameter 0) (color 0 0 0 0)
-  )
-  (junction (at 215.9 34.29) (diameter 0) (color 0 0 0 0)
-  )
-  (junction (at 93.98 156.21) (diameter 0) (color 0 0 0 0)
-  )
-  (junction (at 203.2 71.12) (diameter 0) (color 0 0 0 0)
-  )
-  (junction (at 132.08 59.69) (diameter 0) (color 0 0 0 0)
   )
   (no_connect (at -43.18 44.45))
@@
     (stroke (width 0) (type default) (color 0 0 0 0))
   )
-  (wire (pts (xy 124.46 156.21) (xy 114.3 156.21))
-    (stroke (width 0) (type default) (color 0 0 0 0))
-  )
   (wire (pts (xy 184.15 80.01) (xy 179.07 80.01))
     (stroke (width 0) (type default) (color 0 0 0 0))
@@
     (stroke (width 0) (type default) (color 0 0 0 0))
   )
-  (wire (pts (xy 104.14 161.29) (xy 114.3 161.29))
-    (stroke (width 0) (type default) (color 0 0 0 0))
-  )
   (wire (pts (xy 132.08 64.77) (xy 132.08 67.31))
     (stroke (width 0) (type default) (color 0 0 0 0))
@@
     (stroke (width 0) (type default) (color 0 0 0 0))
   )
-  (wire (pts (xy 114.3 161.29) (xy 124.46 161.29))
-    (stroke (width 0) (type default) (color 0 0 0 0))
-  )
   (wire (pts (xy 132.08 54.61) (xy 132.08 57.15))
     (stroke (width 0) (type default) (color 0 0 0 0))
@@
   )
   (wire (pts (xy 184.15 64.77) (xy 179.07 64.77))
-    (stroke (width 0) (type default) (color 0 0 0 0))
-  )
-  (wire (pts (xy 114.3 156.21) (xy 104.14 156.21))
     (stroke (width 0) (type default) (color 0 0 0 0))
   )
@@
     )
     (property "Datasheet" "~" (id 3) (at 104.14 158.75 0)
-      (effects (font (size 1.27 1.27)) hide)
-    )
-    (pin "1")
-    (pin "2")
-  )
-  (symbol (lib_id "Device:C_Small") (at 114.3 158.75 0) (unit 1)
-    (in_bom yes) (on_board yes)
-    (property "Reference" "C5" (id 0) (at 116.6368 157.5816 0)
-      (effects (font (size 1.27 1.27)) (justify left))
-    )
-    (property "Value" "2u2" (id 1) (at 116.6368 159.893 0)
-      (effects (font (size 1.27 1.27)) (justify left))
-    )
-    (property "Footprint" "stdpads:C_0805" (id 2) (at 114.3 158.75 0)
-      (effects (font (size 1.27 1.27)) hide)
-    )
-    (property "Datasheet" "~" (id 3) (at 114.3 158.75 0)
       (effects (font (size 1.27 1.27)) hide)
     )
@@
     (pin "1")
   )
-  (symbol (lib_id "power:GND") (at 124.46 161.29 0) (unit 1)
-    (in_bom yes) (on_board yes)
-    (property "Reference" "#PWR?" (id 0) (at 124.46 167.64 0)
-      (effects (font (size 1.27 1.27)) hide)
-    )
-    (property "Value" "GND" (id 1) (at 124.46 165.1 0))
-    (property "Footprint" "" (id 2) (at 124.46 161.29 0)
-      (effects (font (size 1.27 1.27)) hide)
-    )
-    (property "Datasheet" "" (id 3) (at 124.46 161.29 0)
-      (effects (font (size 1.27 1.27)) hide)
-    )
-    (pin "1")
-  )
-  (symbol (lib_id "Device:C_Small") (at 124.46 158.75 0) (unit 1)
-    (in_bom yes) (on_board yes)
-    (property "Reference" "C6" (id 0) (at 126.7968 157.5816 0)
-      (effects (font (size 1.27 1.27)) (justify left))
-    )
-    (property "Value" "2u2" (id 1) (at 126.7968 159.893 0)
-      (effects (font (size 1.27 1.27)) (justify left))
-    )
-    (property "Footprint" "stdpads:C_0805" (id 2) (at 124.46 158.75 0)
-      (effects (font (size 1.27 1.27)) hide)
-    )
-    (property "Datasheet" "~" (id 3) (at 124.46 158.75 0)
-      (effects (font (size 1.27 1.27)) hide)
-    )
-    (pin "1")
-    (pin "2")
+  (symbol (lib_id "power:GND") (at 104.14 161.29 0) (unit 1)
+    (in_bom yes) (on_board yes)
+    (property "Reference" "#PWR0110" (id 0) (at 104.14 167.64 0)
+      (effects (font (size 1.27 1.27)) hide)
+    )
+    (property "Value" "GND" (id 1) (at 104.14 165.1 0))
+    (property "Footprint" "" (id 2) (at 104.14 161.29 0)
+      (effects (font (size 1.27 1.27)) hide)
+    )
+    (property "Datasheet" "" (id 3) (at 104.14 161.29 0)
+      (effects (font (size 1.27 1.27)) hide)
+    )
+    (pin "1")
   )
   (sheet_instances
@@
       (reference "#PWR0109") (unit 1) (value "+5V") (footprint "")
     )
+    (path "/00000000-0000-0000-0000-000062ea79d6"
+      (reference "#PWR0110") (unit 1) (value "GND") (footprint "")
+    )
     (path "/00000000-0000-0000-0000-000060be1609"
       (reference "#PWR0111") (unit 1) (value "GND") (footprint "")
@@
       (reference "#PWR0113") (unit 1) (value "+5V") (footprint "")
     )
-    (path "/00000000-0000-0000-0000-000062ea79d6"
-      (reference "#PWR?") (unit 1) (value "GND") (footprint "")
-    )
     (path "/00000000-0000-0000-0000-00005c2e290a"
       (reference "C1") (unit 1) (value "2u2") (footprint "stdpads:C_0805")
@@
       (reference "C4") (unit 1) (value "2u2") (footprint "stdpads:C_0805")
     )
-    (path "/00000000-0000-0000-0000-00005d3fc322"
-      (reference "C5") (unit 1) (value "2u2") (footprint "stdpads:C_0805")
-    )
-    (path "/00000000-0000-0000-0000-000062ea79df"
-      (reference "C6") (unit 1) (value "2u2") (footprint "stdpads:C_0805")
-    )
     (path "/00000000-0000-0000-0000-000060bd711b"
